Commit message: vehicle descriptions and control added

File: vehicle_description/urdf/cart_holonomic_files/cart_holonomic_macros.xacro (robot description, xacro)
@@ -19,13 +19,13 @@
           </geometry>
         </collision>
-        <visual name="${name}_visual">
+        <!--visual name="${name}_visual">
           <origin rpy="0 1.5707 1.5707" xyz="0 0 0"/>
           <geometry>
             <cylinder length="0.04" radius="0.1"/>
           </geometry>
-        </visual>
+        </visual-->
     </link>
 </macro>
-<macro name="joint_wheel" params="name child origin_xyz">
+<macro name="joint_wheel" params="name child origin_xyz damping friction">
   <joint name="${name}" type="continuous">
     <origin rpy="0 0 0" xyz="${origin_xyz}"/>
@@ -34,5 +34,15 @@
     <axis rpy="0 0 0" xyz="0 1 0"/>
     <limit effort="10000" velocity="1000"/>
-    <joint_properties damping="1.0" friction="1.0"/>
+    <joint_properties damping="${damping}" friction="${friction}"/>  <!-- <joint_properties damping="1.0" riction="1.0"/>  -->
+  </joint>
+</macro>
+<macro name="fixed_wheel" params="name child origin_xyz damping friction">
+  <joint name="${name}" type="fixed">
+    <origin rpy="0 0 0" xyz="${origin_xyz}"/>
+    <child link="${child}"/>
+    <parent link="link_chassis"/>
+    <axis rpy="0 0 0" xyz="0 1 0"/>
+    <limit effort="10000" velocity="1000"/>
+    <joint_properties damping="${damping}" friction="${friction}"/>  <!-- <joint_properties damping="1.0" riction="1.0"/>  -->
   </joint>
 </macro>

File: vehicle_description/urdf/castor.xacro (robot description, xacro)
@@ -1,7 +1,7 @@
 <?xml version="1.0" ?>
 <robot name="castor" xmlns:xacro="http://www.ros.org/wiki/xacro">
-  <xacro:include filename="$(find vehicle_description)/urdf/castor_materials.xacro" />
-  <xacro:include filename="$(find vehicle_description)/urdf/castor.gazebo" />
-  <xacro:include filename="$(find vehicle_description)/urdf/castor_macros.xacro" />
+  <xacro:include filename="$(find vehicle_description)/urdf/castor_files/castor_materials.xacro" />
+  <xacro:include filename="$(find vehicle_description)/urdf/castor_files/castor.gazebo" />
+  <xacro:include filename="$(find vehicle_description)/urdf/castor_files/castor_macros.xacro" />
   <link name="link_chassis">
     <!-- pose and inertial -->
