Commit message: added nadir camera

File: rotors_simulator/rotors_description/urdf/firefly_base.xacro (robot description, xacro)
@@ -41,3 +41,22 @@
       wait_to_record_bag="$(arg wait_to_record_bag)" />
   </xacro:if>
+   <!--Mount a Camera-->
+   <!-- Copied from https://github.com/ethz-asl/rotors_simulator/wiki/Adding-a-Camera-to-RotorS  -->
+  <xacro:camera_macro
+    namespace="${namespace}"
+    parent_link="${namespace}/base_link"
+    camera_suffix="nadir"
+    frame_rate="20.0"
+    horizontal_fov="2"
+    image_width="752"
+    image_height="480"
+    image_format="L8"
+    min_distance="0.02"
+    max_distance="50"
+    noise_mean="0.0"
+    noise_stddev="0.007"
+    enable_visual="true">
+    <box size="0.05 0.05 0.02" />
+    <origin xyz="0 0 ${-arm_length/4}" rpy="0 ${pi/2} 0" />
+  </xacro:camera_macro>
 </robot>
