Commit message: added new message to stop motors and made urdf file read the mesh file successfully: changed needed for visual and collision blocks

File: rotors_simulator/rotors_description/urdf/multirotor_base.xacro (robot description, xacro)
@@ -62,4 +62,16 @@
           <box size="${body_width} ${body_width} ${body_height}" /> <!-- [m] [m] [m] -->
         </geometry>
+        <!--  hardik: friction added  -->
+        <surface>
+          <friction>
+            <ode>
+              <mu>0.9</mu>
+              <mu2>0.9</mu2>
+              <slip1>0.0</slip1>
+            <slip2>0.0</slip2>
+            </ode>
+          </friction>
+        </surface>
+        <!--    -->
       </collision>
     </link>

File: vehicle_description/urdf/cart_holonomic.xacro (robot description, xacro)
@@ -1,4 +1,4 @@
 <?xml version="1.0" ?>
-<robot name="castor" xmlns:xacro="http://www.ros.org/wiki/xacro">
+<robot name="ambulance" xmlns:xacro="http://www.ros.org/wiki/xacro">
   <xacro:include filename="$(find vehicle_description)/urdf/cart_holonomic_files/cart_holonomic_materials.xacro" />
   <xacro:include filename="$(find vehicle_description)/urdf/cart_holonomic_files/cart_holonomic.gazebo" />
@@ -7,82 +7,33 @@
   <link name="base_footprint">
   <visual>
-      <origin xyz="0 0 0" rpy="0 0 0" />
+      <origin xyz="0 0 0" rpy="0 0 1.57" />
+      <!--geometry>
+        <box size="2.0 2.0 0.25" />
+      </geometry-->
       <geometry>
-        <box size="2.0 2.0 0.25" />
+            <mesh filename="/media/hardik/Windows/Ubuntu/catkin_740/src/AE740_FINAL_PROJECT/vehicle_description/ambulance/meshes/ambulance.obj" scale="0.0254 0.0254 0.0254"/>
       </geometry>
-    </visual>
+   </visual>
    <collision>
-      <origin xyz="0 0 0" rpy="0 0 0" />
+      <origin xyz="0 0 1.7" rpy="0 0 0" />
       <geometry>
-        <box size="2.0 2.0 0.25" />
+        <box size="6.0 2.9 2.9" /> <!--box size="2.0 2.0 0.25" /-->
       </geometry>
-    </collision>
-    <inertial>
-      <mass value="50"/>
-      <origin rpy="0 0 0" xyz="0 0 0"/>
-      <inertia ixx="1.0" ixy="0" ixz="0" iyy="1.0" iyz="0" izz="2.0"/>
-    </inertial>
-     <surface>
+           <surface>
         <friction>
           <ode>
-            <mu>0.5</mu>
-            <mu2>0.5</mu2>
-            <slip1>0.3</slip1>
-            <slip2>0.3</slip2>
+            <mu>1.0</mu>
+            <mu2>1.0</mu2>
+            <slip1>0</slip1>
+            <slip2>0</slip2>
           </ode>
         </friction>
       </surface>
-  </link>
-  <joint name="base_link_joint" type="fixed">
-    <origin xyz="0.0 0 0" rpy="0 0 0" />
-    <parent link="base_footprint"/>
-    <child link="link_chassis" />
-  </joint>
-  <link name="link_chassis">
-    <!-- pose and inertial -->
-    <pose>0 0 0.1 0 0 0</pose>
-    <!--inertial>
-      <mass value="5"/>
+    </collision>
+    <inertial>
+      <mass value="3000"/>
       <origin rpy="0 0 0" xyz="0 0 0"/>
-      <inertia ixx="0.0395416666667" ixy="0" ixz="0" iyy="0.106208333333" iyz="0" izz="0.106208333333"/>
-    </inertial-->
-    <!-- body -->
-    <visual>
-      <origin rpy="0 0 0" xyz="0 0 0"/>
-      <geometry>
-        <box size="2.0 2.0 0.07"/>
-      </geometry>
-      <material name="blue"/>
-    </visual>
-    <!-- front wheels only for visual -->
-    <visual name="left_front_wheel">
-      <origin rpy="0 1.5707 1.5707" xyz="1.0 -1.0 0"/>
-      <geometry>
-            <cylinder length="0.04" radius="0.1"/>
-      </geometry>
-      <material name="white"/>
-    </visual>
-    <visual name="right_front_wheel">
-      <origin rpy="0 1.5707 1.5707" xyz="1.0 1.0 0"/>
-      <geometry>
-            <cylinder length="0.04" radius="0.1"/>
-      </geometry>
-      <material name="white"/>
-    </visual>
-    <!-- rear wheels only for visual -->
-    <visual name="left_rear_wheel">
-      <origin rpy="0 1.5707 1.5707" xyz="-1.0 -1.0 0"/>
-      <geometry>
-            <cylinder length="0.04" radius="0.1"/>
-      </geometry>
-      <material name="blue"/>
-    </visual>
-    <visual name="right_rear_wheel">
-      <origin rpy="0 1.5707 1.5707" xyz="-1.0 1.0 0"/>
-      <geometry>
-            <cylinder length="0.04" radius="0.1"/>
-      </geometry>
-      <material name="blue"/>
-    </visual>
+      <inertia ixx="1000.0" ixy="0" ixz="0" iyy="1000.0" iyz="0" izz="2000.0"/>
+    </inertial>
   </link>
 </robot>

File: vehicle_description/urdf/cart_unicycle.xacro (robot description, xacro)
@@ -34,6 +34,6 @@
         <friction>
           <ode>
-            <mu>0</mu>
-            <mu2>0</mu2>
+            <mu>0.9</mu>
+            <mu2>0.9</mu2>
             <slip1>1.0</slip1>
             <slip2>1.0</slip2>
