Commit message: hopping drone achieved [successful]

File: vehicle_description/urdf/cart_holonomic.xacro (robot description, xacro)
@@ -6,8 +6,14 @@
   <!-- invisible root link, on the ground just below the model origin -->
   <link name="base_footprint">
+  <visual>
+      <origin xyz="0 0 0" rpy="0 0 0" />
+      <geometry>
+        <box size="2.0 2.0 0.25" />
+      </geometry>
+    </visual>
    <collision>
       <origin xyz="0 0 0" rpy="0 0 0" />
       <geometry>
-        <box size="0.5 0.3 0.25" />
+        <box size="2.0 2.0 0.25" />
       </geometry>
     </collision>
@@ -45,5 +51,5 @@
       <origin rpy="0 0 0" xyz="0 0 0"/>
       <geometry>
-        <box size="0.5 0.3 0.07"/>
+        <box size="2.0 2.0 0.07"/>
       </geometry>
       <material name="blue"/>
@@ -51,5 +57,5 @@
     <!-- front wheels only for visual -->
     <visual name="left_front_wheel">
-      <origin rpy="0 1.5707 1.5707" xyz="0.2 -0.2 0"/>
+      <origin rpy="0 1.5707 1.5707" xyz="1.0 -1.0 0"/>
       <geometry>
             <cylinder length="0.04" radius="0.1"/>
@@ -58,5 +64,5 @@
     </visual>
     <visual name="right_front_wheel">
-      <origin rpy="0 1.5707 1.5707" xyz="0.2 0.2 0"/>
+      <origin rpy="0 1.5707 1.5707" xyz="1.0 1.0 0"/>
       <geometry>
             <cylinder length="0.04" radius="0.1"/>
@@ -66,5 +72,5 @@
     <!-- rear wheels only for visual -->
     <visual name="left_rear_wheel">
-      <origin rpy="0 1.5707 1.5707" xyz="-0.2 -0.2 0"/>
+      <origin rpy="0 1.5707 1.5707" xyz="-1.0 -1.0 0"/>
       <geometry>
             <cylinder length="0.04" radius="0.1"/>
@@ -73,5 +79,5 @@
     </visual>
     <visual name="right_rear_wheel">
-      <origin rpy="0 1.5707 1.5707" xyz="-0.2 0.2 0"/>
+      <origin rpy="0 1.5707 1.5707" xyz="-1.0 1.0 0"/>
       <geometry>
             <cylinder length="0.04" radius="0.1"/>

Commit message: fixed so that visual and collision block coincide but friction in Y < friction in X

File: vehicle_description/urdf/cart_holonomic.xacro (robot description, xacro)
@@ -16,5 +16,5 @@
    </visual>
    <collision>
-      <origin xyz="0 0 1.7" rpy="0 0 0" />
+      <origin xyz="0 0 1.45" rpy="0 0 0" />   <!-- this makes it float way above in air -->
       <geometry>
         <box size="6.0 2.9 2.9" /> <!--box size="2.0 2.0 0.25" /-->

Commit message: modified file path

File: vehicle_description/urdf/cart_holonomic.xacro (robot description, xacro)
@@ -12,5 +12,5 @@
       </geometry-->
       <geometry>
-            <mesh filename="/media/hardik/Windows/Ubuntu/catkin_740/src/AE740_FINAL_PROJECT/vehicle_description/ambulance/meshes/ambulance.obj" scale="0.0254 0.0254 0.0254"/>
+            <mesh filename="$(find vehicle_description)/ambulance/meshes/ambulance.obj" scale="0.0254 0.0254 0.0254"/>
       </geometry>
    </visual>

Commit message: improvements

File: vehicle_description/urdf/cart_holonomic.xacro (robot description, xacro)
@@ -8,9 +8,12 @@
   <visual>
       <origin xyz="0 0 0" rpy="0 0 1.57" />
-      <!--geometry>
-        <box size="2.0 2.0 0.25" />
-      </geometry-->
       <geometry>
             <mesh filename="$(find vehicle_description)/ambulance/meshes/ambulance.obj" scale="0.0254 0.0254 0.0254"/>
+      </geometry>
+   </visual>
+   <visual>
+      <origin xyz="-3.0 0 3.0" rpy="0 0 1.57" />
+      <geometry>
+            <box size="2.5 0.1 0.25" />
       </geometry>
    </visual>
@@ -31,4 +34,10 @@
       </surface>
     </collision>
+    <collision>
+    <origin xyz="-3.0 0 3.0" rpy="0 0 1.57" />
+      <geometry>
+            <box size="2.5 0.1 0.25" />
+      </geometry>
+    </collision>
     <inertial>
       <mass value="3000"/>

Commit message: FINSIHED

File: vehicle_description/urdf/cart_holonomic.xacro (robot description, xacro)
@@ -12,10 +12,10 @@
       </geometry>
    </visual>
-   <visual>
+   <!-- <visual>
       <origin xyz="-3.0 0 3.0" rpy="0 0 1.57" />
       <geometry>
             <box size="2.5 0.1 0.25" />
       </geometry>
-   </visual>
+   </visual> -->
    <collision>
       <origin xyz="0 0 1.45" rpy="0 0 0" />   <!-- this makes it float way above in air -->
@@ -34,10 +34,10 @@
       </surface>
     </collision>
-    <collision>
+    <!-- <collision>
     <origin xyz="-3.0 0 3.0" rpy="0 0 1.57" />
       <geometry>
             <box size="2.5 0.1 0.25" />
       </geometry>
-    </collision>
+    </collision> -->
     <inertial>
       <mass value="3000"/>
